Commit message: Working trajectories, position control and servoing

File: description/urdf/arm_description.urdf.xacro (robot description, xacro)
@@ -123,5 +123,5 @@
     <joint name="joint_4" type="revolute">
         <axis xyz="0 0 1"/>
-        <limit effort="1000.0" lower="-3.927" upper="3.927" velocity="0.5"/>
+        <limit effort="1000.0" lower="-6.4" upper="6.4" velocity="0.5"/>
         <parent link="link3"/>
         <child link="link4"/>
@@ -213,5 +213,6 @@
         <parent link="link5_ext"/>
         <child link="link6"/>
-        <origin rpy="0 0 0" xyz="0.01 0.01 0.0"/>
+        <!-- <origin rpy="0 0 0" xyz="0.02 0.0 0.0"/> -->
+        <origin rpy="0 0 0" xyz="0.0 0.0 0.0"/>
     </joint>
     <joint name="joint_6_to_gripper" type="fixed" >

File: description/urdf/dupsko.urdf (robot description, URDF)
Before this commit: robot arm, 15 links, 14 joints
Joints:
- joint joint_4: limit lower=-3.927 upper=3.927 effort=1000.0 velocity=0.5 -> lower=-6.4 upper=6.4 effort=1000.0 velocity=0.5
- joint joint_6: origin xyz=0.01 0.01 0.0 rpy=0 0 0 -> xyz=-0.02 0.02 0.0 rpy=0 0 0
