Commit message: Working collision detection on servo

File: description/urdf/arm.urdf.xacro (robot description, xacro)
@@ -7,4 +7,24 @@
         <child link="flange" />
     </joint>
+    <joint name="fix_colision" type="fixed">
+        <parent link="world" />
+        <child link="kalman_box" />
+    </joint>
+    <link name="kalman_box">
+        <visual>
+            <geometry>
+                <!-- <mesh filename="package://kalman_arm_controller/meshes/gripper/gripper_bottom.stl" scale="0.001 0.001 0.001"/> -->
+                <box size="1.0 1.0 0.1"/>
+            </geometry>
+        <origin rpy="0 0 0" xyz="-0.04 -0.04 -0.12"/>
+        <material name="white"/>1
+        </visual>
+        <collision>
+            <geometry>
+                <box size="1.0 1.0 0.1"/>
+            </geometry>
+        <origin rpy="0 0 0" xyz="-0.04 -0.04 -0.12"/>
+        </collision>
+    </link>
     <xacro:include filename="$(find kalman_arm_controller)/urdf/arm_description.urdf.xacro"/>
     <xacro:arm_description />

File: description/urdf/dupsko.urdf (robot description, URDF)
Before this commit: robot arm, 15 links, 14 joints
Links:
- added link kalman_box; collision box size=1.0 1.0 0.1; visual box size=1.0 1.0 0.1
Joints:
- added joint fix_colision: type fixed, parent world, child kalman_box
